File: kicad/K24LR1MA_m88_rangefinder.kicad_sch (KiCad schematic)
At the start: 52 parts, among them J1 Conn_01x08_Socket, J2 Conn_01x08_Socket, J3 Conn_01x04_Socket, J4 Conn_01x04_Socket, J5 USB_C_Receptacle_USB2.0 USB41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, J6 Conn_01x04_Socket, Q1 DMG3402L, Q2 DMG3402L, SW5 SW_Push, SW6 SW_SPST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

Commit message: added 5v converter capacitors
Parts:
- added C15, C16: 100n, Capacitor_SMD:C_0603_1608Metric, symbol Device:C
- added C3, C4: 10u, Capacitor_SMD:C_0603_1608Metric, symbol Device:C
- added J7: Conn_01x02_Pin, Connector_PinHeader_2.54mm:PinHeader_1x02_P2.54mm_Vertical, symbol Connector:Conn_01x02_Pin
- D1: value D_Schottky -> SD103AWS; footprint (none) -> Diode_SMD:D_SOD-323
Connections:
- net +5V: now also D1.1 (K), R17.2, C16.2, C4.2
- net +BATT: now also C15.2, C3.2, J7.1 (Pin_1)
- net GND: now also C15.1, C16.1, C3.1, C4.1
- net GND1: now also J7.2 (Pin_2)
Other:
- note added: "HC-SR04"
- note added: "LASER"
- note added: "OLED"
- moved on the sheet: BT1, D1, L1, R17, R18, U5
